Commit message: added lidar

File: description/robot.urdf.xacro (robot description, xacro)
@@ -1,4 +1,5 @@
 <?xml version="1.0"?>
-<robot name="bot_v3">
+<robot xmlns:xacro="http://www.ros.org/wiki/xacro" name="robot">
+    <xacro:include filename= "lidar.xacro"/>
   <material name="green_dark">
     <color rgba="0.0 0.5 0.0 1"/>
@@ -20,21 +21,21 @@
   <!-- Body -->
   <link name="chassis">
-    <visual>
-      <geometry>
-        <box size="0.1 0.075 0.03"/>
-      </geometry>
-      <material name="box_bot_blue"/>
-    </visual>
+     <visual>
+        <geometry>
+          <box size="0.1 0.075 0.03"/>
+        </geometry>
+        <material name="box_bot_blue"/>
+     </visual>
   <inertial>
-      <mass value="0.2"/>
-      <origin rpy="0 0 0" xyz="0 0 0"/>
-      <inertia ixx= "0.00010875"  ixy= "0" ixz= "0" iyy= "0.0001816666666666667" iyz= "0" izz= "0.0001816666666666667" />
+    <mass value="0.2"/>
+    <origin rpy="0 0 0" xyz="0 0 0"/>
+    <inertia ixx= "0.00010875"  ixy= "0" ixz= "0" iyy= "0.0001816666666666667" iyz= "0" izz= "0.0001816666666666667" />
   </inertial>
   <collision>
-      <geometry>
-        <box size="0.1 0.075 0.03"/>
-      </geometry>
+    <geometry>
+      <box size="0.1 0.075 0.03"/>
+    </geometry>
   </collision>
-  </link>
+</link>
   <gazebo reference="chassis">
       <material>Gazebo/Blue</material>
@@ -221,122 +222,3 @@
     </plugin>
   </gazebo>
-  <link name="rgb_camera_link_frame">
-    <visual>
-      <origin rpy="0 0 0" xyz="0 0 0"/>
-      <geometry>
-        <box size="0.02 0.02 0.02"/>
-      </geometry>
-    </visual>
-    <collision>
-       <origin rpy="0 0 0" xyz="0 0 0.0204"/>
-      <geometry>
-        <box size="0.02 0.02 0.02"/>
-      </geometry>
-    </collision>
-    <inertial>
-      <mass value="0.01"/>
-      <origin rpy="0 0 0" xyz="0 0 0.0204"/>
-      <inertia ixx="6.066578520833334e-06" ixy="0" ixz="0" iyy="6.072950163333333e-06" iyz="0" izz="9.365128684166666e-06"/>
-    </inertial>
-  </link>
-  <joint name="rgb_camera_link_frame_joint" type="fixed">
-      <origin rpy="0.0 0.2 3.1416" xyz="-0.045 0.0 0.001"/>
-      <parent link="chassis" />
-      <child link="rgb_camera_link_frame" />
-      <axis xyz="0 0 0"/>
-  </joint>
-     <gazebo reference="rgb_camera_link_frame">
-        <sensor name="camera" type="camera">
-            <visualize>true</visualize>
-            <pose>0 0 0 0 0.2 0</pose>
-            <update_rate>30.0</update_rate>
-            <always_on>1</always_on>
-            <camera name="camera">
-                <horizontal_fov>1.3962634</horizontal_fov>
-                <image>
-                    <width>480</width>
-                    <height>360</height>
-                    <format>R8G8B8</format>
-                </image>
-                <clip>
-                    <!-- distance described in meters -->
-                    <near>0.01</near>
-                    <far>300</far>
-                </clip>
-                <distortion>
-                    <k1>0.0</k1>
-                    <k2>0.0</k2>
-                    <k3>0.0</k3>
-                    <p1>0.0</p1>
-                    <p2>0.0</p2>
-                    <center>0.5 0.5</center>
-                </distortion>
-            </camera>
-            <plugin filename="libgazebo_ros_camera.so" name="camera_controller">
-            <ros>
-                <remapping>~/image_raw:=camera/image</remapping>
-                <remapping>~/camera_info:=camera/camera_info</remapping>
-            </ros>
-            <frame_name>rgb_camera_link_frame</frame_name>
-            </plugin>
-        </sensor>
-    </gazebo>
-<link name="lidar_link">
-  <visual>
-    <origin xyz="0 0 -0.030" rpy="0 0 0"/>
-    <geometry>
-      <cylinder length="0.015" radius="0.02"/>
-    </geometry>
-    <material name="yellow"/>
-  </visual>
-  <collision>
-    <origin xyz="0 0 -0.0150" rpy="0 0 0"/>
-    <geometry>
-      <cylinder length="0.015" radius="0.02"/>
-    </geometry>
-  </collision>
-  <inertial>
-    <mass value="0.1"/>
-    <origin xyz="0 0 0" rpy="0 0 0"/>
-    <inertia ixx="0.0001" ixy="0" ixz="0" iyy="0.0001" iyz="0" izz="0.0001"/>
-  </inertial>
-</link>
-<joint name="lidar_joint" type="fixed">
-  <origin xyz="0 0 0.05" rpy="0 0 0"/>
-  <parent link="chassis"/>
-  <child link="lidar_link"/>
-</joint>
-<gazebo reference="lidar_link">
-  <sensor name="laser" type="ray">
-    <pose>0 0 0 0 0 0</pose>
-    <visualize>true</visualize>
-    <update_rate>20</update_rate>
-    <ray>
-      <scan>
-        <horizontal>
-          <samples>720</samples>
-          <resolution>1</resolution>
-          <min_angle>-1.5708</min_angle>
-          <max_angle>1.5708</max_angle>
-        </horizontal>
-      </scan>
-      <range>
-        <min>0.12</min>
-        <max>3.5</max>
-        <resolution>0.01</resolution>
-      </range>
-      <noise>
-        <type>gaussian</type>
-        <mean>0.0</mean>
-        <stddev>0.01</stddev>
-      </noise>
-    </ray>
-    <plugin name="gazebo_ros_laser_controller" filename="libgazebo_ros_laser.so">
-      <ros>
-        <remapping>~/scan:=scan</remapping>
-      </ros>
-      <frame_name>lidar_link</frame_name>
-    </plugin>
-  </sensor>
-</gazebo>
 </robot>

File: description/robot_core.xacro (robot description, xacro)
@@ -1,4 +1,5 @@
 <?xml version="1.0"?>
 <robot xmlns:xacro="http://www.ros.org/wiki/xacro"  >
+    <xacro:include filename="inertial_macros.xacro" />
     <!-- <xacro:include filename ="robot_core.xacro" /> -->
     <material name="white">
@@ -29,4 +30,54 @@
             <material name="white"/>
         </visual>
+        <collision>
+            <origin xyz="0.15 0 0.075" rpy="0 0 0"/>
+            <geometry>
+                <box size="0.3 0.3 0.15"/>
+            </geometry>
+        </collision>
+    </link>
+<!-- LEFT WHEEL -->
+    <joint name="left_wheel_joint" type="continuous">
+        <parent link="base_link"/>
+        <child link="left_wheel"/>
+        <origin xyz="0 0.175 0" rpy="-${pi/2} 0 0"/>
+        <axis xyz="0 0 1"/>
+    </joint>
+    <link name="left_wheel">
+        <visual>
+            <geometry>
+                <cylinder length="0.04" radius="0.05" />
+            </geometry>
+            <material name="blue"/>
+        </visual>
+    </link>
+    <!-- RIGHT WHEEL -->
+    <joint name="right_wheel_joint" type="continuous">
+        <parent link="base_link"/>
+        <child link="right_wheel"/>
+        <origin xyz="0 -0.175 0" rpy="${pi/2} 0 0"/>
+        <axis xyz="0 0 -1"/>
+    </joint>
+    <link name="right_wheel">
+        <visual>
+            <geometry>
+                <cylinder length="0.04" radius="0.05" />
+            </geometry>
+            <material name="blue"/>
+        </visual>
+    </link>
+    <!-- CASTER WHEEL -->
+    <joint name="caster_wheel_joint" type="fixed">
+        <parent link="chassis"/>
+        <child link="caster_wheel"/>
+        <origin xyz="0.24 0 0" rpy="0 0 0"/>
+    </joint>
+    <link name="caster_wheel">
+        <visual>
+            <geometry>
+                <sphere radius="0.05" />
+            </geometry>
+            <material name="black"/>
+        </visual>
     </link>
 </robot>
